File: yuiop27.kicad_pcb (KiCad board)
At the start: 2 copper layers, 147.6 x 97.6 mm, 90 parts, among them J1 MJ-4PP-9, SW1 SW_PUSH, SW10 SW_PUSH, SW11 SW_PUSH, SW12 SW_PUSH, SW13 SW_PUSH, SW14 SW_PUSH, SW15 SW_PUSH, SW16 SW_PUSH, SW17 SW_PUSH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

Commit message: make references unique
Parts:
- removed REF** (x4): MountingHole_4.3mm_M4, MountingHole:MountingHole_4.3mm_M4
- added REF01: MountingHole_4.3mm_M4, MountingHole:MountingHole_4.3mm_M4, F.Cu at (100.8, 83.4)
- added REF02: MountingHole_4.3mm_M4, MountingHole:MountingHole_4.3mm_M4, F.Cu at (201.6, 76.5)
- added REF03: MountingHole_4.3mm_M4, MountingHole:MountingHole_4.3mm_M4, F.Cu at (162.8, 100.8)
- added REF04: MountingHole_4.3mm_M4, MountingHole:MountingHole_4.3mm_M4, F.Cu at (196.8, 127.0)
- renumbered REF** to REF05
Changed lines of the file:
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@@
     (tags "mounting hole 4.3mm no annular m4")
     (attr virtual)
-    (fp_text reference REF** (at 0 -5.3) (layer F.SilkS) hide
+    (fp_text reference REF01 (at 0 -5.3) (layer F.SilkS) hide
       (effects (font (size 1 1) (thickness 0.15)))
     )
@@
     (tags "mounting hole 4.3mm no annular m4")
     (attr virtual)
-    (fp_text reference REF** (at 0 -5.3) (layer F.SilkS) hide
+    (fp_text reference REF02 (at 0 -5.3) (layer F.SilkS) hide
       (effects (font (size 1 1) (thickness 0.15)))
     )
@@
     (tags "mounting hole 4.3mm no annular m4")
     (attr virtual)
-    (fp_text reference REF** (at 0 -5.3) (layer F.SilkS) hide
+    (fp_text reference REF03 (at 0 -5.3) (layer F.SilkS) hide
       (effects (font (size 1 1) (thickness 0.15)))
     )
@@
     (tags "mounting hole 4.3mm no annular m4")
     (attr virtual)
-    (fp_text reference REF** (at 0 -5.3) (layer F.SilkS) hide
+    (fp_text reference REF04 (at 0 -5.3) (layer F.SilkS) hide
       (effects (font (size 1 1) (thickness 0.15)))
     )
@@
     (tags "mounting hole 4.3mm no annular m4")
     (attr virtual)
-    (fp_text reference REF** (at 0 -5.3) (layer F.SilkS) hide
+    (fp_text reference REF05 (at 0 -5.3) (layer F.SilkS) hide
       (effects (font (size 1 1) (thickness 0.15)))
     )
