File: yuiop54/yuiop54-w0.kicad_pcb (KiCad board)
At the start: 2 copper layers, 285 x 94.6 mm, 173 parts, among them SW1 SW_PUSH, SW10 SW_PUSH, SW11 SW_PUSH, SW12 SW_PUSH, SW13 SW_PUSH, SW14 SW_PUSH, SW15 SW_PUSH, SW16 SW_PUSH, SW17 SW_PUSH, SW18 SW_PUSH, SW19 SW_PUSH, SW2 SW_PUSH, SW20 SW_PUSH, SW21 SW_PUSH, SW22 SW_PUSH, SW23 SW_PUSH, SW24 SW_PUSH, SW25 SW_PUSH, SW26 SW_PUSH, SW27 SW_PUSH, SW28 SW_PUSH, SW29 SW_PUSH, SW3 SW_PUSH, SW30 SW_PUSH, SW31 SW_PUSH, SW32 SW_PUSH, SW33 SW_PUSH, SW34 SW_PUSH, SW35 SW_PUSH, SW36 SW_PUSH, SW37 SW_PUSH, SW38 SW_PUSH, SW39 SW_PUSH, SW4 SW_PUSH, SW40 SW_PUSH, SW41 SW_PUSH, SW42 SW_PUSH, SW43 SW_PUSH, SW44 SW_PUSH, SW45 SW_PUSH, SW46 SW_PUSH, SW47 SW_PUSH, SW48 SW_PUSH, SW49 SW_PUSH, SW5 SW_PUSH, SW50 SW_PUSH, SW51 SW_PUSH, SW52 SW_PUSH, SW53 SW_PUSH, SW54 SW_PUSH, SW6 SW_PUSH, SW7 SW_PUSH, SW8 SW_PUSH, SW9 SW_PUSH, U1 ProMicro

Commit message: wired YUIOP55
Routing:
- net VCC: track 1720.0 -> 0.00 mm, vias 28 -> 0
- net GND: track 1697.9 -> 0.00 mm, vias 24 -> 0
- net COL6: track 326.3 -> 0.00 mm, vias 11 -> 0
- net COL1: track 319.9 -> 0.00 mm, vias 10 -> 0
- net COL2: track 307.0 -> 0.00 mm, vias 11 -> 0
- net COL3: track 304.7 -> 0.00 mm, vias 11 -> 0
- net COL5: track 302.2 -> 0.00 mm, vias 11 -> 0
- net COL4: track 300.4 -> 0.00 mm, vias 11 -> 0
- net ROW9: track 220.8 -> 0.00 mm, vias 3 -> 0
- net LED: track 187.3 -> 0.00 mm
- net ROW8: track 166.3 -> 0.00 mm, vias 1 -> 0
- net ROW7: track 164.1 -> 0.00 mm, vias 1 -> 0
- net ROW4: track 161.5 -> 0.00 mm
- net ROW3: track 158.0 -> 0.00 mm, vias 1 -> 0
- net ROW5: track 153.3 -> 0.00 mm
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Other:
- rule trace_min: 0 -> 0.2
