File: yuiop54/yuiop54.sch (KiCad schematic (older format))
At the start: 166 parts, among them SW1 SW_PUSH, SW10 SW_PUSH, SW11 SW_PUSH, SW12 SW_PUSH, SW13 SW_PUSH, SW14 SW_PUSH, SW15 SW_PUSH, SW16 SW_PUSH, SW17 SW_PUSH, SW18 SW_PUSH, SW19 SW_PUSH, SW2 SW_PUSH, SW20 SW_PUSH, SW21 SW_PUSH, SW22 SW_PUSH, SW23 SW_PUSH, SW24 SW_PUSH, SW25 SW_PUSH, SW26 SW_PUSH, SW27 SW_PUSH, SW28 SW_PUSH, SW29 SW_PUSH, SW3 SW_PUSH, SW30 SW_PUSH, SW31 SW_PUSH, SW32 SW_PUSH, SW33 SW_PUSH, SW34 SW_PUSH, SW35 SW_PUSH, SW36 SW_PUSH, SW37 SW_PUSH, SW38 SW_PUSH, SW39 SW_PUSH, SW4 SW_PUSH, SW40 SW_PUSH, SW41 SW_PUSH, SW42 SW_PUSH, SW43 SW_PUSH, SW44 SW_PUSH, SW45 SW_PUSH, SW46 SW_PUSH, SW47 SW_PUSH, SW48 SW_PUSH, SW49 SW_PUSH, SW5 SW_PUSH, SW50 SW_PUSH, SW51 SW_PUSH, SW52 SW_PUSH, SW53 SW_PUSH, SW54 SW_PUSH, SW6 SW_PUSH, SW7 SW_PUSH, SW8 SW_PUSH, SW9 SW_PUSH, U1 ProMicro

Commit message: wired YUIOP55
Parts:
- SW1, SW10, SW11, SW12, SW14, SW15, SW16, SW17, SW18, SW19, SW2, SW20, SW21, SW22, SW23, SW26, SW27, SW28, SW29, SW3, SW30, SW31, SW32, SW33, SW34, SW35, SW38, SW39, SW4, SW40, SW41, SW42, SW43, SW44, SW45, SW46, SW47, SW5, SW6, SW7, SW8, SW9: footprint kbd:CherryMX_Hotswap -> yuiop:Cherry_MX_Hotswap_1u
- SW49: footprint kbd:CherryMX_Hotswap -> yuiop:Cherry_MX_Hotswap_1.25u
Connections:
- net COL2: now also SW53.1
- net COL3: now also SW54.1
- net COL4: now also U1.18 (F6/A1); no longer U1.7 (4/D4)
- net COL5: now also U1.7 (4/D4); no longer U1.18 (F6/A1)
- net COL6: now also U1.17 (F7/A0); no longer U1.8 (5/C6)
- net ROW1: now also U1.8 (5/C6); no longer U1.17 (F7/A0)
- net ROW2: now also U1.16 (B1/15); no longer U1.9 (6/D7)
- net ROW3: now also U1.9 (6/D7); no longer U1.16 (B1/15)
- net ROW4: now also U1.15 (B3/14); no longer U1.10 (7/E6)
- net ROW5: now also U1.10 (7/E6); no longer U1.15 (B3/14)
- net ROW6: now also U1.14 (B2/16); no longer U1.11 (8/B4)
- net ROW7: now also U1.11 (8/B4); no longer SW53.1, SW54.1, U1.14 (B2/16)
- net ROW8: now also U1.13 (B6/10); no longer U1.12 (9/B5)
- net ROW9: now also U1.12 (9/B5); no longer U1.13 (B6/10)
Other:
- moved on the sheet: LED1, LED10, LED11, LED12, LED13, LED14, LED15, LED16, LED17, LED18, LED19, LED2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
