File: yuiop54/yuiop54.kicad_pcb (KiCad board)
At the start: 2 copper layers, 285 x 94.6 mm, 173 parts, among them SW1 SW_PUSH, SW10 SW_PUSH, SW11 SW_PUSH, SW12 SW_PUSH, SW13 SW_PUSH, SW14 SW_PUSH, SW15 SW_PUSH, SW16 SW_PUSH, SW17 SW_PUSH, SW18 SW_PUSH, SW19 SW_PUSH, SW2 SW_PUSH, SW20 SW_PUSH, SW21 SW_PUSH, SW22 SW_PUSH, SW23 SW_PUSH, SW24 SW_PUSH, SW25 SW_PUSH, SW26 SW_PUSH, SW27 SW_PUSH, SW28 SW_PUSH, SW29 SW_PUSH, SW3 SW_PUSH, SW30 SW_PUSH, SW31 SW_PUSH, SW32 SW_PUSH, SW33 SW_PUSH, SW34 SW_PUSH, SW35 SW_PUSH, SW36 SW_PUSH, SW37 SW_PUSH, SW38 SW_PUSH, SW39 SW_PUSH, SW4 SW_PUSH, SW40 SW_PUSH, SW41 SW_PUSH, SW42 SW_PUSH, SW43 SW_PUSH, SW44 SW_PUSH, SW45 SW_PUSH, SW46 SW_PUSH, SW47 SW_PUSH, SW48 SW_PUSH, SW49 SW_PUSH, SW5 SW_PUSH, SW50 SW_PUSH, SW51 SW_PUSH, SW52 SW_PUSH, SW53 SW_PUSH, SW54 SW_PUSH, SW6 SW_PUSH, SW7 SW_PUSH, SW8 SW_PUSH, SW9 SW_PUSH, U1 ProMicro

Commit message: replace by auto routing version
Routing:
- net VCC: track 1720.0 -> 1316.4 mm, vias 28 -> 2
- net GND: track 1697.9 -> 1425.7 mm, vias 24 -> 1
- net ROW6: track 151.2 -> 202.4 mm, vias 0 -> 3
- net ROW1: track 137.4 -> 176.2 mm, vias 1 -> 3
- net ROW5: track 153.3 -> 188.7 mm, vias 0 -> 4
- net LED: track 187.3 -> 155.9 mm, vias 0 -> 1
- net COL1: track 319.9 -> 349.3 mm, vias 10 -> 2
- net ROW2: track 136.4 -> 159.7 mm, vias 1 -> 3
- net Net-(LED30-Pad2): track 34.3 -> 57.0 mm, vias 2 -> 0
- net COL6: track 326.3 -> 345.2 mm, vias 11 -> 1
- net COL4: track 300.4 -> 318.7 mm, vias 11 -> 6
- net Net-(LED25-Pad2): track 41.3 -> 25.3 mm, vias 2 -> 0
- net Net-(LED7-Pad2): track 37.5 -> 22.3 mm, vias 2 -> 0
- net Net-(LED34-Pad2): track 36.1 -> 21.8 mm, vias 2 -> 0
- net Net-(LED15-Pad2): track 35.0 -> 21.3 mm, vias 2 -> 0
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Other:
- rule trace_min: 0 -> 0.2
