File: yuiop27/yuiop27.kicad_pcb (KiCad board)
At the start: 2 copper layers, 147.6 x 97.6 mm, 90 parts, among them J1 MJ-4PP-9, SW1 SW_PUSH, SW10 SW_PUSH, SW11 SW_PUSH, SW12 SW_PUSH, SW13 SW_PUSH, SW14 SW_PUSH, SW15 SW_PUSH, SW16 SW_PUSH, SW17 SW_PUSH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

Commit message: update yuiop27
Parts:
- OL1: footprint kbd:OLED_1side -> yuiop:OLED_128x32
- SW13: footprint kbd:CherryMX_Hotswap -> yuiop:Cherry_MX_Hotswap_1.75u
- SW19, SW26, SW27: footprint kbd:CherryMX_Hotswap -> yuiop:Cherry_MX_Hotswap_1.25u
- SW25, SW7: footprint kbd:CherryMX_Hotswap -> yuiop:Cherry_MX_Hotswap_1.5u
- moved OL1 3.88 mm to (214.0, 98.4)
- turned SW13 to 0 degrees
- turned SW19 to 0 degrees
- turned SW25 to 0 degrees
- turned SW26 to 0 degrees
- turned SW27 to 90 degrees
- turned SW7 to 0 degrees
Routing:
- added copper zone on B.Cu, net GND
- added copper zone on F.Cu, net GND
