File: yuiop60hh2/yuiop60hh2.kicad_pcb (KiCad board)
At the start: 2 copper layers, 285 x 94.6 mm, 183 parts, among them SW1 SW_PUSH, SW10 SW_PUSH, SW11 SW_PUSH, SW12 SW_PUSH, SW13 SW_PUSH, SW14 SW_PUSH, SW15 SW_PUSH, SW16 SW_PUSH, SW17 SW_PUSH, SW18 SW_PUSH, SW19 SW_PUSH, SW2 SW_PUSH, SW20 SW_PUSH, SW21 SW_PUSH, SW22 SW_PUSH, SW23 SW_PUSH, SW24 SW_PUSH, SW25 SW_PUSH, SW26 SW_PUSH, SW27 SW_PUSH, SW28 SW_PUSH, SW29 SW_PUSH, SW3 SW_PUSH, SW30 SW_PUSH, SW31 SW_PUSH, SW32 SW_PUSH, SW33 SW_PUSH, SW34 SW_PUSH, SW35 SW_PUSH, SW36 SW_PUSH, SW37 SW_PUSH, SW38 SW_PUSH, SW39 SW_PUSH, SW4 SW_PUSH, SW40 SW_PUSH, SW41 SW_PUSH, SW42 SW_PUSH, SW43 SW_PUSH, SW44 SW_PUSH, SW45 SW_PUSH, SW46 SW_PUSH, SW47 SW_PUSH, SW48 SW_PUSH, SW49 SW_PUSH, SW5 SW_PUSH, SW50 SW_PUSH, SW51 SW_PUSH, SW52 SW_PUSH, SW53 SW_PUSH, SW54 SW_PUSH, SW55 SW_PUSH, SW56 SW_PUSH, SW57 SW_PUSH, SW58 SW_PUSH, SW59 SW_PUSH, SW6 SW_PUSH, SW60 SW_PUSH, SW7 SW_PUSH, SW8 SW_PUSH, SW9 SW_PUSH, U1 ProMicro

Commit message: yuiop60hh/2 auto wired
Routing:
- net GND: track 0.00 -> 1446.9 mm, vias 0 -> 41
- net VCC: track 0.00 -> 1394.5 mm, vias 0 -> 4
- net /COL5: track 0.00 -> 535.0 mm, vias 0 -> 4
- net /COL3: track 0.00 -> 494.2 mm, vias 0 -> 6
- net /COL2: track 0.00 -> 455.4 mm, vias 0 -> 6
- net /COL8: track 0.00 -> 433.3 mm, vias 0 -> 5
- net /COL7: track 0.00 -> 387.6 mm, vias 0 -> 3
- net /COL4: track 0.00 -> 379.5 mm, vias 0 -> 8
- net /COL6: track 0.00 -> 372.5 mm, vias 0 -> 5
- net /ROW1: track 0.00 -> 372.4 mm, vias 0 -> 1
- net /LED: track 0.00 -> 363.6 mm
- net /COL1: track 0.00 -> 361.1 mm, vias 0 -> 5
- net /ROW2: track 0.00 -> 354.5 mm, vias 0 -> 2
- net /ROW3: track 0.00 -> 306.2 mm, vias 0 -> 4
- net /ROW4: track 0.00 -> 260.4 mm, vias 0 -> 2
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- added copper zone on B.Cu, net GND
- added copper zone on F.Cu, net GND
