File: yuiop60hh3/yuiop60hh3.kicad_pcb (KiCad board)
At the start: 2 copper layers, 285 x 94.6 mm, 159 parts, among them J1 USB_B_Micro, J2 ISP, U1 ATmega32U4-AU, X1 XTAL

Commit message: yuiop60hh3: finish top plate, generate gerbers
Routing:
- net /ROW_3: track 423.3 -> 424.6 mm
- net /COL_03: track 129.5 -> 130.3 mm
- net GND: track 606.1 -> 606.5 mm, vias 1 -> 4
- added copper zone on F.Cu, net GND
Other:
- board text added: "GND"
- board text added: "JLCJLCJLCJLC"
- board text added: "MISO"
- board text added: "MOSI"
- board text added: "RESET"
- board text added: "SCLK"
- board text added: "VCC"
- board text added: "YUIOP60HH3"
- board text added: "designed by KoRoN/KaoriYa"
