File: yuiop60hh3-r2/controller.sch (KiCad schematic (older format))
At the start: 18 parts, among them J1 USB_B_Micro, J2 ISP, U1 ATmega32U4-AU, X1 XTAL

Commit message: yuiop60hh3-r2: beta finish
Parts:
- removed J1: USB_B_Micro, KeyboardController:USB-MicroB_ZX62M-B-5P, symbol Connector:USB_B_Micro
- removed J2: ISP, Connector_PinHeader_2.54mm:PinHeader_2x03_P2.54mm_Vertical, symbol Connector_Generic:Conn_02x03_Odd_Even
Connections:
- net USB_VBUS: now reaches F1.2
- net USB_D-: now reaches R4.2
- net USB_D+: now reaches R3.2
- net P09_B1_SCLK renamed P09_B1
- net P10_B2_MOSI renamed P10_B2
- net P11_B3_MISO renamed P11_B3
- no-connect marks 2 -> 1
Other:
- moved on the sheet: C1, C2, D0, F1, R1, R3, R4, X1
