File: yuiop60hh3-r2/leds.sch (KiCad schematic (older format))
At the start: 5 parts

Commit message: yuiop60hh3-r2: beta finish
Parts:
- LED1, LED2, LED3, LED4, LED5: footprint LED_SMD:LED_SK6812MINI_PLCC4_3.5x3.5mm_P1.75mm -> yuiop:SK6812MINI-E_B; symbol LED:SK6812MINI -> kbd:YS-SK6812MINI-E
Connections:
- net DIN: now also LED1.4 (DIN); no longer LED1.3 (DIN)
- net DOUT: now also LED5.2 (DOUT); no longer LED5.1 (DOUT)
- net VDD: now also LED1.1 (VDD), LED2.1 (VDD), LED3.1 (VDD), LED4.1 (VDD), LED5.1 (VDD); no longer LED1.4 (VDD), LED2.4 (VDD), LED3.4 (VDD), LED4.4 (VDD), LED5.4 (VDD)
- net VSS: now also LED1.3 (VSS), LED2.3 (VSS), LED3.3 (VSS), LED4.3 (VSS), LED5.3 (VSS); no longer LED1.2 (VSS), LED2.2 (VSS), LED3.2 (VSS), LED4.2 (VSS), LED5.2 (VSS)
- new net: LED1.2 (DOUT), LED2.4 (DIN)
- new net: LED2.2 (DOUT), LED3.4 (DIN)
- new net: LED3.2 (DOUT), LED4.4 (DIN)
- new net: LED4.2 (DOUT), LED5.4 (DIN)
Changed lines of the file:
@@
 $EndDescr
 $Comp
-L LED:SK6812MINI LED1
+L kbd:YS-SK6812MINI-E LED1
 U 1 1 60709497
 P 4475 4025
 F 0 "LED1" H 4525 4275 50  0000 L CNN
 F 1 "SK6812MINI" H 4500 3775 50  0000 L CNN
-F 2 "LED_SMD:LED_SK6812MINI_PLCC4_3.5x3.5mm_P1.75mm" H 4525 3725 50  0001 L TNN
+F 2 "yuiop:SK6812MINI-E_B" H 4525 3725 50  0001 L TNN
 F 3 "https://cdn-shop.adafruit.com/product-files/2686/SK6812MINI_REV.01-1-2.pdf" H 4575 3650 50  0001 L TNN
 	1    4475 4025
@@
 $EndComp
 $Comp
-L LED:SK6812MINI LED2
+L kbd:YS-SK6812MINI-E LED2
 U 1 1 60710D9B
 P 5225 4025
 F 0 "LED2" H 5275 4275 50  0000 L CNN
 F 1 "SK6812MINI" H 5250 3775 50  0000 L CNN
-F 2 "LED_SMD:LED_SK6812MINI_PLCC4_3.5x3.5mm_P1.75mm" H 5275 3725 50  0001 L TNN
+F 2 "yuiop:SK6812MINI-E_B" H 5275 3725 50  0001 L TNN
 F 3 "https://cdn-shop.adafruit.com/product-files/2686/SK6812MINI_REV.01-1-2.pdf" H 5325 3650 50  0001 L TNN
 	1    5225 4025
@@
 $EndComp
 $Comp
-L LED:SK6812MINI LED3
+L kbd:YS-SK6812MINI-E LED3
 U 1 1 60714963
 P 5975 4025
 F 0 "LED3" H 6025 4275 50  0000 L CNN
 F 1 "SK6812MINI" H 6000 3775 50  0000 L CNN
-F 2 "LED_SMD:LED_SK6812MINI_PLCC4_3.5x3.5mm_P1.75mm" H 6025 3725 50  0001 L TNN
+F 2 "yuiop:SK6812MINI-E_B" H 6025 3725 50  0001 L TNN
 F 3 "https://cdn-shop.adafruit.com/product-files/2686/SK6812MINI_REV.01-1-2.pdf" H 6075 3650 50  0001 L TNN
 	1    5975 4025
@@
 $EndComp
 $Comp
-L LED:SK6812MINI LED4
+L kbd:YS-SK6812MINI-E LED4
 U 1 1 60714969
 P 6725 4025
 F 0 "LED4" H 6775 4275 50  0000 L CNN
 F 1 "SK6812MINI" H 6750 3775 50  0000 L CNN
-F 2 "LED_SMD:LED_SK6812MINI_PLCC4_3.5x3.5mm_P1.75mm" H 6775 3725 50  0001 L TNN
+F 2 "yuiop:SK6812MINI-E_B" H 6775 3725 50  0001 L TNN
 F 3 "https://cdn-shop.adafruit.com/product-files/2686/SK6812MINI_REV.01-1-2.pdf" H 6825 3650 50  0001 L TNN
 	1    6725 4025
@@
 $EndComp
 $Comp
-L LED:SK6812MINI LED5
+L kbd:YS-SK6812MINI-E LED5
 U 1 1 607167DB
 P 7475 4025
 F 0 "LED5" H 7525 4275 50  0000 L CNN
 F 1 "SK6812MINI" H 7500 3775 50  0000 L CNN
-F 2 "LED_SMD:LED_SK6812MINI_PLCC4_3.5x3.5mm_P1.75mm" H 7525 3725 50  0001 L TNN
+F 2 "yuiop:SK6812MINI-E_B" H 7525 3725 50  0001 L TNN
 F 3 "https://cdn-shop.adafruit.com/product-files/2686/SK6812MINI_REV.01-1-2.pdf" H 7575 3650 50  0001 L TNN
 	1    7475 4025
