File: yuiop60hh3-r2/yuiop60hh3-r2-topplate.kicad_pcb (KiCad board)
At the start: 2 copper layers, 285 x 94.6 mm, 75 parts

Commit message: yuiop60hh3-r2: beta finish
Parts:
- HOLE10, HOLE11, HOLE12, HOLE7, HOLE8, HOLE9: value Hole_2.2_4 -> H3.5mm spacer
- moved HOLE11 19.3 mm to (222.0, 113.4)
- moved HOLE7 19.3 mm to (126.8, 113.4)
- moved HOLE12 5.21 mm to (207.7, 170.3)
- moved HOLE10 5.21 mm to (332.6, 170.3)
- moved HOLE8 5.21 mm to (110.0, 170.3)
- moved HOLE9 4.91 mm to (317.3, 113.4)
- moved 1 4.14 mm to (314.5, 185.4)
- moved 2 2.58 mm to (323.1, 185.4)
- moved 5 2.16 mm to (348.8, 185.4)
- moved 3 1.04 mm to (331.7, 185.4)
- moved 4 0.65 mm to (340.2, 185.4)
- moved KSW43 0.49 mm to (91.1, 166.4)
- moved KSW44 0.49 mm to (122.0, 166.4)
- moved KSW45 0.49 mm to (141.1, 166.4)
- moved KSW46 0.49 mm to (160.1, 166.4)
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Other:
- outline, holes or cut-outs redrawn
