File: yuiop60hh3-r2/yuiop60hh3-r2.kicad_pcb (KiCad board)
At the start: 2 copper layers, 285 x 94.6 mm, 159 parts, among them J1 USB_B_Micro, J2 ISP, U1 ATmega32U4-AU, X1 XTAL

Commit message: yuiopPM: biuld guide
Routing:
- net /Controller/D-: track 108.6 -> 103.2 mm
- net GND: track 622.2 -> 619.6 mm, vias 3 -> 1
- net /LED_DATA: track 147.2 -> 149.2 mm
- net VCC: track 366.8 -> 365.6 mm

Commit message: yuiop60hh3-r2: beta finish
Parts:
- J1: footprint KeyboardController:USB-MicroB_ZX62M-B-5P -> Connector_USB:USB_Micro-B_Amphenol_10103594-0001LF_Horizontal
- LED1, LED2, LED3, LED4, LED5: footprint LED_SMD:LED_SK6812MINI_PLCC4_3.5x3.5mm_P1.75mm -> yuiop:SK6812MINI-E_B
- moved J2 78.4 mm to (226.7, 182.1)
- moved R2 29.3 mm to (161.3, 190.0), turned to 0 degrees
- moved C2 28.2 mm to (189.8, 187.6)
- moved C1 26.4 mm to (189.8, 179.6), turned to 0 degrees
- moved C6 24.5 mm to (161.3, 186.2), turned to 180 degrees
- moved R3 23.6 mm to (103.3, 164.8)
- moved R4 23.3 mm to (103.3, 168.1)
- moved X1 22.5 mm to (189.8, 183.7), turned to 0 degrees
- moved R1 20.5 mm to (183.9, 178.6), turned to 180 degrees
- moved HOLE11 19.3 mm to (222.0, 113.4)
- moved HOLE7 19.3 mm to (126.8, 113.4), turned to 180 degrees
- moved C3 18.6 mm to (183.9, 189.8), turned to 0 degrees
- moved D56 16.6 mm to (117.2, 187.8)
- moved D58 16.6 mm to (212.5, 187.8)
- moved D59 16.6 mm to (283.9, 187.8)
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Connections:
- net Net-(F1-Pad2) renamed /USB_VBUS
- net Net-(J1-Pad2) renamed /USB_D-
- net Net-(J1-Pad3) renamed /USB_D+
- HOLE3 pad : (no net) -> GND
- J2 pad 1: /Controller/P11_B3_MISO -> /LED_DATA
- J2 pad 3: /Controller/P09_B1_SCLK -> /COL_07
- J2 pad 4: /Controller/P10_B2_MOSI -> /COL_08
- LED1 pad 1: Net-(LED1-Pad1) -> VCC
- LED1 pad 2: GND -> Net-(LED1-Pad2)
- LED1 pad 3: /LED_DATA -> GND
- LED1 pad 4: VCC -> /LED_DATA
- LED2 pad 1: Net-(LED2-Pad1) -> VCC
- LED2 pad 2: GND -> Net-(LED2-Pad2)
- LED2 pad 3: Net-(LED1-Pad1) -> GND
- LED2 pad 4: VCC -> Net-(LED1-Pad2)
- LED3 pad 1: Net-(LED3-Pad1) -> VCC
- LED3 pad 2: GND -> Net-(LED3-Pad2)
- LED3 pad 3: Net-(LED2-Pad1) -> GND
- LED3 pad 4: VCC -> Net-(LED2-Pad2)
- LED4 pad 1: Net-(LED4-Pad1) -> VCC
- LED4 pad 2: GND -> Net-(LED4-Pad2)
- LED4 pad 3: Net-(LED3-Pad1) -> GND
- LED4 pad 4: VCC -> Net-(LED3-Pad2)
- LED5 pad 1: /LED Array/DOUT -> VCC
- LED5 pad 2: GND -> /LED Array/DOUT
- LED5 pad 3: Net-(LED4-Pad1) -> GND
- LED5 pad 4: VCC -> Net-(LED4-Pad2)
- U1 pad 1: /LED_DATA -> /Controller/P01_E6
- U1 pad 10: /Controller/P10_B2_MOSI -> /COL_08
- U1 pad 11: /Controller/P11_B3_MISO -> /LED_DATA
- U1 pad 12: /COL_02 -> /Controller/P12_B7
- U1 pad 18: /COL_03 -> /Controller/P18_D0
- U1 pad 19: /COL_04 -> /COL_09
- U1 pad 20: /COL_05 -> /COL_10
- U1 pad 21: /COL_06 -> /COL_11
- U1 pad 22: /COL_07 -> /COL_12
- U1 pad 25: /COL_08 -> /COL_13
- U1 pad 26: /COL_09 -> /COL_14
- U1 pad 27: /COL_10 -> /COL_15
- U1 pad 28: /COL_11 -> /COL_01
- U1 pad 29: /COL_12 -> /COL_02
- U1 pad 30: /COL_13 -> /COL_03
- U1 pad 31: /COL_14 -> /COL_04
- U1 pad 32: /COL_15 -> /COL_05
- U1 pad 8: /COL_01 -> /COL_06
- U1 pad 9: /Controller/P09_B1_SCLK -> /COL_07
Routing:
- net /COL_07: track 127.6 -> 206.8 mm, vias 3 -> 0
- net /COL_08: track 125.2 -> 187.5 mm, vias 0 -> 1
- net /RESET: track 104.1 -> 153.8 mm, vias 1 -> 2
- net GND: track 619.6 -> 654.9 mm
- net VCC: track 365.6 -> 334.5 mm, vias 3 -> 7
- net /Controller/P09_B1_SCLK: track 29.6 -> 0.00 mm
- net /Controller/D-: track 103.2 -> 73.8 mm, vias 0 -> 2
- net /Controller/P10_B2_MOSI: track 29.1 -> 0.00 mm
- net /COL_12: track 232.8 -> 205.7 mm
- net /COL_02: track 142.7 -> 169.0 mm, vias 3 -> 0
- net /ROW_5: track 212.5 -> 186.5 mm, vias 3 -> 4
- net /Controller/P11_B3_MISO: track 25.2 -> 0.00 mm, vias 1 -> 0
- net /ROW_4: track 379.1 -> 354.0 mm, vias 8 -> 7
- net /COL_09: track 135.8 -> 159.7 mm
- net /COL_05: track 80.7 -> 103.5 mm
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- added copper zone on B.Cu, net GND
Other:
- outline, holes or cut-outs redrawn
- net class Power added: clearance 0.2, trace_width 0.4, via_dia 0.8, via_drill 0.4
