File: yuiop60hh3-r2/yuiop60hh3-r2.sch (KiCad schematic (older format))
At the start: 1 part

Commit message: yuiop60hh3-r2: beta finish
Parts:
- added J1: USB_B_Micro, Connector_USB:USB_Micro-B_Amphenol_10103594-0001LF_Horizontal, symbol Connector:USB_B_Micro
- added J2: ISP, Connector_PinHeader_2.54mm:PinHeader_2x03_P2.54mm_Vertical, symbol Connector_Generic:Conn_02x03_Odd_Even
Connections:
- net GND: now also J2.6 (Pin_6)
- net RESET: now also J2.5 (Pin_5)
- net VCC: now also J2.2 (Pin_2)
- new net MISO: J2.1 (Pin_1)
- new net MOSI: J2.4 (Pin_4)
- new net SCLK: J2.3 (Pin_3)
- new net USB_D+: J1.3 (D+)
- new net USB_D-: J1.2 (D-)
- new net USB_GND: J1.5 (GND), J1.6 (Shield)
- new net USB_VBUS: J1.1 (VBUS)
- no-connect marks 2 -> 6
Other:
- moved on the sheet: RSW1
