File: yuiop60hh4/yuiop60hh4-topplate.kicad_pcb (KiCad board)
At the start: 2 copper layers, 285 x 94.6 mm, 75 parts

Commit message: rename to yuiop60hh4 <- yuiop60hh3-r2
Other:
- board text added: "YUIOP60HH"
- board text added: "revision 4"
- board text removed: "YUIOP60HH3"
- board text removed: "revision 2"
Changed lines of the file:
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@@
   (page A3)
   (title_block
-    (title YUIOP60HH3)
-    (date 2021-04-21)
-    (rev 2)
+    (title "YUIOP60HH/Top plate")
+    (date 2021-04-22)
+    (rev 4)
     (company KaoriYa)
   )
@@
     (pad_to_mask_clearance 0)
     (aux_axis_origin 70 100)
-    (grid_origin 331.677 185.441)
+    (grid_origin 70 100)
     (visible_elements 7FF7FFFF)
     (pcbplotparams
@@
     (pad "" np_thru_hole circle (at 0 0) (size 4.8 4.8) (drill 4.8) (layers *.Cu *.Mask))
   )
-  (gr_text "revision 2" (at 92.65 187.884) (layer F.SilkS)
+  (gr_text "revision 4" (at 92.5 188) (layer F.SilkS)
     (effects (font (size 1 1) (thickness 0.15)))
   )
@@
     (effects (font (size 0.8 0.8) (thickness 0.15)) (justify mirror))
   )
-  (gr_text "designed by KoRoN/KaoriYa" (at 85.748 189.916) (layer F.SilkS)
+  (gr_text "designed by KoRoN/KaoriYa" (at 85.6 190) (layer F.SilkS)
     (effects (font (size 1 1) (thickness 0.15)))
   )
-  (gr_text YUIOP60HH3 (at 84.85 184.95) (layer F.SilkS)
+  (gr_text YUIOP60HH (at 86 185) (layer F.SilkS)
     (effects (font (size 3.5 2.5) (thickness 0.4)))
   )
