File: yuiop60hh4/yuiop60hh4.kicad_pcb (KiCad board)
At the start: 2 copper layers, 285 x 94.6 mm, 159 parts, among them J1 USB_B_Micro, J2 ISP, U1 ATmega32U4-AU, X1 XTAL

Commit message: rename to yuiop60hh4 <- yuiop60hh3-r2
Other:
- board text added: "YUIOP60HH"
- board text added: "revision 4"
- board text removed: "YUIOP60HH3"
- board text removed: "revision 2"
Changed lines of the file:
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@@
   (page A3)
   (title_block
-    (title YUIOP60HH3)
+    (title YUIOP60HH)
     (date 2021-04-22)
-    (rev 2)
+    (rev 4)
     (company KaoriYa)
   )
@@
     (arrow2b (pts (xy 51.555001 117.89484) (xy 52.141421 119.021343)))
   )
-  (gr_text "revision 2" (at 92.65 187.884) (layer F.SilkS)
+  (gr_text "revision 4" (at 92.5 188) (layer F.SilkS)
     (effects (font (size 1 1) (thickness 0.15)))
   )
@@
     (effects (font (size 0.8 0.8) (thickness 0.15)) (justify mirror))
   )
-  (gr_text "designed by KoRoN/KaoriYa" (at 85.748 189.916) (layer F.SilkS)
+  (gr_text "designed by KoRoN/KaoriYa" (at 85.6 190) (layer F.SilkS)
     (effects (font (size 1 1) (thickness 0.15)))
   )
-  (gr_text YUIOP60HH3 (at 84.85 184.95) (layer F.SilkS)
+  (gr_text YUIOP60HH (at 86 185) (layer F.SilkS)
     (effects (font (size 3.5 2.5) (thickness 0.4)))
   )
