File: yuiop31rs/yuiop31rs.kicad_pcb (KiCad board)
At the start: 2 copper layers, 116.5 x 116.5 mm, 105 parts, among them SW1 SW_PUSH, SW10 SW_PUSH, SW11 SW_PUSH, SW12 SW_PUSH, SW13 SW_PUSH, SW14 SW_PUSH, SW15 SW_PUSH, SW16 SW_PUSH, SW17 SW_PUSH, SW18 SW_PUSH, SW19 SW_PUSH, SW2 SW_PUSH, SW20 SW_PUSH, SW21 SW_PUSH, SW22 SW_PUSH, SW23 SW_PUSH, SW24 SW_PUSH, SW25 SW_PUSH, SW26 SW_PUSH, SW27 SW_PUSH, SW28 SW_PUSH, SW29 SW_PUSH, SW3 SW_PUSH, SW30 SW_PUSH, SW31 SW_PUSH, SW4 SW_PUSH, SW5 SW_PUSH, SW6 SW_PUSH, SW7 SW_PUSH, SW8 SW_PUSH, SW9 SW_PUSH, U1 ProMicro

Commit message: yuiop31rs: fix circuit, generate gerbers
Connections:
- D32 pad 1: Net-(D32-Pad1) -> /ROW_3
- D32 pad 2: /COL_1 -> Net-(D32-Pad2)
- D33 pad 1: Net-(D33-Pad1) -> /ROW_4
- D33 pad 2: /COL_2 -> Net-(D33-Pad2)
- D34 pad 1: Net-(D34-Pad1) -> /ROW_1
- D34 pad 2: /COL_3 -> Net-(D34-Pad2)
- D35 pad 1: Net-(D35-Pad1) -> /ROW_2
- D35 pad 2: /COL_4 -> Net-(D35-Pad2)
- ROT_SW1 pad 1: Net-(D32-Pad1) -> Net-(D32-Pad2)
- ROT_SW1 pad 2: Net-(D33-Pad1) -> Net-(D35-Pad2)
- ROT_SW1 pad 4: Net-(D34-Pad1) -> Net-(D33-Pad2)
- ROT_SW1 pad 8: Net-(D35-Pad1) -> Net-(D34-Pad2)
- U1 pad 1: /LED_DATA -> Net-(U1-Pad1)
- U1 pad 10: /COL_4 -> /ROW_2
- U1 pad 11: /COL_5 -> /ROW_1
- U1 pad 12: /COL_6 -> /LED_DATA
- U1 pad 13: /ROW_1 -> /COL_6
- U1 pad 14: /ROW_2 -> /COL_5
- U1 pad 15: /ROW_3 -> /COL_4
- U1 pad 16: /ROW_4 -> /COL_3
- U1 pad 17: /ROW_5 -> /COL_2
- U1 pad 18: /ROW_6 -> /ROW_5
- U1 pad 19: /RS -> /ROW_6
- U1 pad 20: Net-(U1-Pad20) -> /COL_1
- U1 pad 7: /COL_1 -> /RS
- U1 pad 8: /COL_2 -> /ROW_4
- U1 pad 9: /COL_3 -> /ROW_3
Routing:
- net /COL_5: track 240.3 -> 162.2 mm, vias 4 -> 5
- net /COL_2: track 133.2 -> 89.2 mm, vias 3 -> 2
- net /ROW_4: track 132.8 -> 175.1 mm, vias 1 -> 3
- net VCC: track 672.6 -> 711.6 mm
- net /COL_6: track 195.8 -> 232.8 mm
- net /ROW_3: track 146.4 -> 182.0 mm
- net Net-(LED4-Pad1): track 71.0 -> 38.9 mm
- net /LED_DATA: track 36.3 -> 8.40 mm, vias 1 -> 0
- net Net-(D34-Pad1): track 27.4 -> 0.00 mm
- net /COL_1: track 84.3 -> 58.9 mm
- net Net-(LED7-Pad1): track 39.5 -> 17.2 mm
- net Net-(LED6-Pad1): track 37.6 -> 17.2 mm
- net Net-(LED17-Pad1): track 17.2 -> 37.2 mm
- net Net-(LED16-Pad1): track 17.2 -> 37.2 mm
- net Net-(LED18-Pad1): track 17.3 -> 37.2 mm
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Other:
- board text added: "JLCJLCJLCJLC"
- board text added: "YUIOP31RS"
- board text added: "designed by KoRoN/KaoriYa"
