File: yuiop60pi/yuiop60pi.kicad_pcb (KiCad board)
At the start: 2 copper layers, 285 x 94.6 mm, 187 parts, among them J1 USB_B_Micro, J2 USB_MON, J3 DEBUG, J4 EXT, Q1 BSS138, U1 PGA2040

Commit message: yuiop60pi: move LEDs
Parts:
- moved LED15 0.20 mm to (86.7, 142.7)
- moved LED16 0.20 mm to (112.9, 142.7)
- moved LED17 0.20 mm to (131.9, 142.7)
- moved LED18 0.20 mm to (151.0, 142.7)
- moved LED19 0.20 mm to (170.0, 142.7)
- moved LED20 0.20 mm to (189.1, 142.7)
- moved LED21 0.20 mm to (208.1, 142.7)
- moved LED22 0.20 mm to (227.2, 142.7)
- moved LED23 0.20 mm to (246.2, 142.7)
- moved LED24 0.20 mm to (265.3, 142.7)
- moved LED25 0.20 mm to (284.3, 142.7)
- moved LED26 0.20 mm to (303.4, 142.7)
- moved LED27 0.20 mm to (334.3, 142.7)
- moved LED28 0.20 mm to (341.5, 123.6)
- moved LED29 0.20 mm to (317.6, 123.6)
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
Commit message: yuiop60pi: wiring, design work
Parts:
- added HOLE1: Hole_5x2.3_6, yuiop:Hole_5x2.5_7, F.Cu at (95.2, 127.9)
- added HOLE10: Hole_2.2_4, yuiop:Hole_2.2_4, F.Cu at (110.0, 165.3)
- added HOLE11: Hole_2.2_4, yuiop:Hole_2.2_4, F.Cu at (207.7, 165.4)
- added HOLE12: Hole_2.2_4, yuiop:Hole_2.2_4, F.Cu at (332.6, 165.3)
- added HOLE2: Hole_5x2.3_6, yuiop:Hole_5x2.5_7, F.Cu at (330.1, 127.9)
- added HOLE3: Hole_2.3, yuiop:Hole_5x2.5_7, F.Cu at (198.2, 147.0)
- added HOLE4: Hole_5x2.3_6, yuiop:Hole_5x2.5_7, F.Cu at (260.5, 185.2)
- added HOLE5: Hole_7x2.5, yuiop:Hole_7x2.5_10x5, F.Cu at (71.5, 156.5)
- added HOLE6: Hole_7x2.5, yuiop:Hole_7x2.5_10x5, F.Cu at (353.5, 156.5)
- added HOLE7: Hole_2.2_4, yuiop:Hole_2.2_4, F.Cu at (126.8, 108.3)
- added HOLE8: Hole_2.2_4, yuiop:Hole_2.2_4, F.Cu at (222.0, 108.3)
- added HOLE9: Hole_2.2_4, yuiop:Hole_2.2_4, F.Cu at (317.3, 108.3)
- added STB2: Cherry_MX_Stabilizer_6.25u, yuiop:Cherry_MX_Stabilizer_6.25u, F.Cu at (200.6, 185.4)
- moved J3 57.2 mm to (314.9, 148.5), turned to 180 degrees
- moved J2 56.3 mm to (286.3, 180.6), turned to 180 degrees
- moved J4 6.09 mm to (345.9, 179.5)
- moved KSW52 0.49 mm to (274.4, 166.4)
- moved KSW59 0.49 mm to (274.4, 185.4)
- moved LED5 0.49 mm to (274.4, 161.4)
- moved D45 0.49 mm to (136.0, 163.8)
- moved D48 0.49 mm to (193.1, 163.8)
- moved D50 0.49 mm to (231.2, 163.8)
- moved KSW46 0.49 mm to (160.1, 166.4)
- moved KSW48 0.49 mm to (198.2, 166.4)
- moved KSW51 0.49 mm to (255.4, 166.4)
- moved LED11 0.49 mm to (160.1, 161.4)
- moved LED6 0.49 mm to (255.4, 161.4)
- moved LED9 0.49 mm to (198.2, 161.4)
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Routing:
- net /GND: track 0.00 -> 1411.4 mm, vias 0 -> 18
- net /VBUS: track 0.00 -> 1217.4 mm, vias 0 -> 2
- net /ROW4: track 0.00 -> 484.3 mm, vias 0 -> 2
- net /ROW1: track 0.00 -> 483.9 mm, vias 0 -> 7
- net /ROW3: track 0.00 -> 386.7 mm, vias 0 -> 7
- net /ROW2: track 0.00 -> 385.0 mm, vias 0 -> 7
- net /USB_D+: track 0.00 -> 309.9 mm, vias 0 -> 1
- net /COL1: track 0.00 -> 296.2 mm
- net /COL2: track 0.00 -> 294.2 mm
- net /USB_D-: track 0.00 -> 284.4 mm, vias 0 -> 1
- net /COL3: track 0.00 -> 272.0 mm
- net /ROW5: track 0.00 -> 258.8 mm, vias 0 -> 1
- net /COL4: track 0.00 -> 239.2 mm, vias 0 -> 1
- net /COL9: track 0.00 -> 237.7 mm
- net /BOOTSEL: track 0.00 -> 232.8 mm, vias 0 -> 1
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- added copper zone on B.Cu, net /GND
- added copper zone on F.Cu, net /GND
Other:
- net class Power added: clearance 0.2, trace_width 0.4, via_dia 0.8, via_drill 0.4
- board text added: "JLCJLCJLCJLC"
- board text added: "YUIOP60Pi"
- board text added: "designed by KoRoN/KaoriYa"
- board text added: "revision 1"
