File: yuiop60pi/main2/main2.kicad_pcb (KiCad board)
At the start: 2 copper layers, 285 x 94.6 mm, 206 parts, among them J1 USB_B_Micro, J2 USB_MON, J3 DEBUG, J4 UART, Q1 BSS138, U1 PGA2040

Commit message: yuiop60pi: plot gerber files for rev 1.2
Other:
- rule trace_min: 0 -> 0.2
