File: yuiop60pi/main3/main3.kicad_pcb (KiCad board)
At the start: 2 copper layers, 285 x 94.6 mm, 206 parts, among them J1 USB_B_Micro, J2 USB_MON, J3 DEBUG, J4 UART, Q1 BSS138, U1 PGA2040

Commit message: wired
Parts:
- moved J3 109.4 mm to (213.1, 187.9), turned to 0 degrees
- moved J4 88.1 mm to (245.0, 182.7)
- moved C1 26.3 mm to (306.6, 172.0)
- moved C3 17.2 mm to (74.8, 147.9), turned to 180 degrees
- moved D59 11.5 mm to (279.5, 188.0)
- moved D60 11.5 mm to (303.3, 188.0)
- moved D57 11.4 mm to (134.3, 188.0)
- moved D58 11.4 mm to (205.7, 188.0)
- moved D56 11.4 mm to (112.8, 188.0)
- moved R1 4.56 mm to (338.9, 182.0)
- moved Q1 4.37 mm to (338.9, 184.8)
- moved DS1 4.30 mm to (143.3, 182.3)
- moved F1 4.30 mm to (143.3, 186.4)
- moved R2 4.18 mm to (338.9, 187.7), turned to 180 degrees
- moved J2 0.91 mm to (157.2, 188.0)
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Routing:
- net /GND: track 2416.2 -> 3033.5 mm, vias 11 -> 7
- net /SWCLK: track 30.3 -> 105.7 mm
- net /SWDIO: track 36.9 -> 105.0 mm, vias 0 -> 1
- net /GPIO1: track 12.1 -> 78.5 mm, vias 0 -> 1
- net /GPIO0: track 12.4 -> 74.2 mm, vias 0 -> 1
- net /VBUS: track 189.7 -> 135.8 mm
- net /COL8: track 174.2 -> 215.2 mm, vias 0 -> 1
- net /COL7: track 218.2 -> 256.9 mm, vias 0 -> 1
- net /COL9: track 161.3 -> 197.6 mm
- net /ROW5: track 250.9 -> 218.2 mm, vias 3 -> 0
- net /COL4: track 241.6 -> 273.8 mm, vias 1 -> 2
- net /COL5: track 224.1 -> 251.6 mm, vias 1 -> 2
- net /BOOTSEL: track 233.5 -> 259.0 mm
- net /COL3: track 276.1 -> 300.9 mm
- net /COL2: track 290.2 -> 314.4 mm
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Other:
- board text added: "revision 3"
- board text removed: "revision 1.2"

Commit message: yuiop60pi/3: brush up
Parts:
- moved J3 24.4 mm to (188.7, 186.7)
- moved J4 1.27 mm to (245.0, 181.4)
Routing:
- net /GND: track 3033.5 -> 2962.8 mm
- net /SWCLK: track 105.7 -> 132.8 mm
- net /SWDIO: track 105.0 -> 130.5 mm
- net /COL4: track 273.8 -> 272.7 mm
- net /USB_D+: track 288.3 -> 287.4 mm
- net /USB_D-: track 288.3 -> 287.4 mm
- net /BOOTSEL: track 259.0 -> 258.1 mm
- net /GPIO0: track 74.2 -> 73.7 mm
- net /GPIO1: track 78.5 -> 78.0 mm
- net /ROW5: track 218.2 -> 217.7 mm

Commit message: add QR code
Parts:
- added G1: LOGO, project:QR_README, B.Cu at (86.5, 183.5)
