File: yuiop60hh/main5/controller.kicad_sch (KiCad schematic)
At the start: 16 parts, among them U1 ATmega32U4-AU, X1 XTAL

Commit message: YUIOP60HH rev.5: finished
Connections:
- net VCC: no longer C7.1, U1.2 (UVCC)
- net V_USB: now also C7.1, U1.2 (UVCC)
Changed lines of the file:
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@@
   (title_block
     (title "YUIOP60HH/Controller")
-    (date "2021-04-22")
-    (rev "4")
+    (date "2022-02-05")
+    (rev "5")
     (company "KaoriYa")
   )
@@
     (stroke (width 0) (type default) (color 0 0 0 0))
   )
-  (label "VCC" (at 142.24 90.17 0)
+  (label "V_USB" (at 142.24 90.17 0)
     (effects (font (size 1.27 1.27)) (justify left bottom))
   )
