File: yuiop60hh/main5/leds.kicad_sch (KiCad schematic)
At the start: 5 parts

Commit message: YUIOP60HH rev.5: finished
Parts:
- removed LED4, LED5: SK6812MINI, yuiop:SK6812MINI-E_B, symbol kbd:YS-SK6812MINI-E
Connections:
- net DOUT: now also LED3.2 (DOUT)
Changed lines of the file:
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@@
   (title_block
     (title "YUIOP60HH/LED Array")
-    (date "2021-04-22")
-    (rev "4")
+    (date "2022-02-05")
+    (rev "5")
     (company "KaoriYa")
   )
@@
   (junction (at 113.665 94.615) (diameter 0) (color 0 0 0 0)
   )
-  (junction (at 151.765 109.855) (diameter 0) (color 0 0 0 0)
-  )
-  (junction (at 170.815 94.615) (diameter 0) (color 0 0 0 0)
-  )
   (junction (at 132.715 109.855) (diameter 0) (color 0 0 0 0)
   )
   (junction (at 132.715 94.615) (diameter 0) (color 0 0 0 0)
-  )
-  (junction (at 170.815 109.855) (diameter 0) (color 0 0 0 0)
-  )
-  (junction (at 151.765 94.615) (diameter 0) (color 0 0 0 0)
   )
   (wire (pts (xy 100.965 102.235) (xy 106.045 102.235))
@@
     (stroke (width 0) (type default) (color 0 0 0 0))
   )
-  (wire (pts (xy 202.565 102.235) (xy 197.485 102.235))
-    (stroke (width 0) (type default) (color 0 0 0 0))
-  )
   (wire (pts (xy 100.965 94.615) (xy 113.665 94.615))
-    (stroke (width 0) (type default) (color 0 0 0 0))
-  )
-  (wire (pts (xy 151.765 109.855) (xy 170.815 109.855))
     (stroke (width 0) (type default) (color 0 0 0 0))
   )
@@
     (stroke (width 0) (type default) (color 0 0 0 0))
   )
-  (wire (pts (xy 182.245 102.235) (xy 178.435 102.235))
-    (stroke (width 0) (type default) (color 0 0 0 0))
-  )
   (wire (pts (xy 132.715 94.615) (xy 151.765 94.615))
     (stroke (width 0) (type default) (color 0 0 0 0))
@@
     (stroke (width 0) (type default) (color 0 0 0 0))
   )
-  (wire (pts (xy 170.815 94.615) (xy 189.865 94.615))
-    (stroke (width 0) (type default) (color 0 0 0 0))
-  )
   (wire (pts (xy 100.965 109.855) (xy 113.665 109.855))
-    (stroke (width 0) (type default) (color 0 0 0 0))
-  )
-  (wire (pts (xy 170.815 109.855) (xy 189.865 109.855))
     (stroke (width 0) (type default) (color 0 0 0 0))
   )
@@
     (stroke (width 0) (type default) (color 0 0 0 0))
   )
-  (wire (pts (xy 151.765 94.615) (xy 170.815 94.615))
-    (stroke (width 0) (type default) (color 0 0 0 0))
-  )
   (hierarchical_label "VDD" (shape input) (at 100.965 94.615 180)
     (effects (font (size 1.27 1.27)) (justify right))
   )
-  (hierarchical_label "DOUT" (shape output) (at 202.565 102.235 0)
+  (hierarchical_label "DOUT" (shape output) (at 163.195 102.235 0)
     (effects (font (size 1.27 1.27)) (justify left))
   )
@@
       (effects (font (size 1.27 1.27)) (justify left top) hide)
     )
-    (pin "1")
-    (pin "2")
-    (pin "3")
-    (pin "4")
-  )
-  (symbol (lib_id "kbd:YS-SK6812MINI-E") (at 170.815 102.235 0) (unit 1)
-    (in_bom yes) (on_board yes)
-    (property "Reference" "LED4" (id 0) (at 172.085 95.885 0)
-      (effects (font (size 1.27 1.27)) (justify left))
-    )
-    (property "Value" "SK6812MINI" (id 1) (at 171.45 108.585 0)
-      (effects (font (size 1.27 1.27)) (justify left))
-    )
-    (property "Footprint" "yuiop:SK6812MINI-E_B" (id 2) (at 172.085 109.855 0)
-      (effects (font (size 1.27 1.27)) (justify left top) hide)
-    )
-    (property "Datasheet" "https://cdn-shop.adafruit.com/product-files/2686/SK6812MINI_REV.01-1-2.pdf" (id 3) (at 173.355 111.76 0)
-      (effects (font (size 1.27 1.27)) (justify left top) hide)
-    )
-    (pin "1")
-    (pin "2")
-    (pin "3")
-    (pin "4")
-  )
-  (symbol (lib_id "kbd:YS-SK6812MINI-E") (at 189.865 102.235 0) (unit 1)
-    (in_bom yes) (on_board yes)
-    (property "Reference" "LED5" (id 0) (at 191.135 95.885 0)
-      (effects (font (size 1.27 1.27)) (justify left))
-    )
-    (property "Value" "SK6812MINI" (id 1) (at 190.5 108.585 0)
-      (effects (font (size 1.27 1.27)) (justify left))
-    )
-    (property "Footprint" "yuiop:SK6812MINI-E_B" (id 2) (at 191.135 109.855 0)
-      (effects (font (size 1.27 1.27)) (justify left top) hide)
-    )
-    (property "Datasheet" "https://cdn-shop.adafruit.com/product-files/2686/SK6812MINI_REV.01-1-2.pdf" (id 3) (at 192.405 111.76 0)
-      (effects (font (size 1.27 1.27)) (justify left top) hide)
-    )
