File: yuiop60hh/main5/yuiop60hh5.kicad_sch (KiCad schematic)
At the start: 3 parts, among them J1 USB_B_Micro, J2 ISP

Commit message: YUIOP60HH rev.5: finished
Changed lines of the file:
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@@
   (title_block
     (title "YUIOP60HH")
-    (date "2021-04-22")
-    (rev "4")
+    (date "2022-02-05")
+    (rev "5")
     (company "KaoriYa")
   )
@@
     (stroke (width 0) (type default) (color 0 0 0 0))
   )
+  (wire (pts (xy 121.92 55.88) (xy 113.03 55.88))
+    (stroke (width 0) (type default) (color 0 0 0 0))
+  )
+  (wire (pts (xy 121.92 73.66) (xy 113.03 73.66))
+    (stroke (width 0) (type default) (color 0 0 0 0))
+  )
+  (wire (pts (xy 121.92 81.28) (xy 113.03 81.28))
+    (stroke (width 0) (type default) (color 0 0 0 0))
+  )
+  (wire (pts (xy 121.92 60.96) (xy 113.03 60.96))
+    (stroke (width 0) (type default) (color 0 0 0 0))
+  )
+  (wire (pts (xy 83.82 166.37) (xy 91.44 166.37))
+    (stroke (width 0) (type default) (color 0 0 0 0))
+  )
+  (wire (pts (xy 76.2 86.36) (xy 85.09 86.36))
+    (stroke (width 0) (type default) (color 0 0 0 0))
+  )
+  (wire (pts (xy 218.44 60.96) (xy 209.55 60.96))
+    (stroke (width 0) (type default) (color 0 0 0 0))
+  )
+  (wire (pts (xy 121.92 97.79) (xy 113.03 97.79))
+    (stroke (width 0) (type default) (color 0 0 0 0))
+  )
+  (wire (pts (xy 74.93 104.14) (xy 85.09 104.14))
+    (stroke (width 0) (type default) (color 0 0 0 0))
+  )
+  (wire (pts (xy 74.93 101.6) (xy 85.09 101.6))
+    (stroke (width 0) (type default) (color 0 0 0 0))
+  )
+  (wire (pts (xy 74.93 66.04) (xy 85.09 66.04))
+    (stroke (width 0) (type default) (color 0 0 0 0))
+  )
+  (wire (pts (xy 218.44 55.88) (xy 209.55 55.88))
+    (stroke (width 0) (type default) (color 0 0 0 0))
+  )
+  (wire (pts (xy 77.47 74.93) (xy 85.09 74.93))
+    (stroke (width 0) (type default) (color 0 0 0 0))
+  )
+  (wire (pts (xy 121.92 88.9) (xy 113.03 88.9))
+    (stroke (width 0) (type default) (color 0 0 0 0))
+  )
+  (wire (pts (xy 83.82 171.45) (xy 91.44 171.45))
+    (stroke (width 0) (type default) (color 0 0 0 0))
+  )
+  (wire (pts (xy 180.34 78.74) (xy 189.23 78.74))
+    (stroke (width 0) (type default) (color 0 0 0 0))
+  )
+  (wire (pts (xy 118.11 135.89) (xy 105.41 135.89))
+    (stroke (width 0) (type default) (color 0 0 0 0))
+  )
+  (wire (pts (xy 180.34 53.34) (xy 189.23 53.34))
+    (stroke (width 0) (type default) (color 0 0 0 0))
+  )
+  (wire (pts (xy 180.34 68.58) (xy 189.23 68.58))
+    (stroke (width 0) (type default) (color 0 0 0 0))
+  )
+  (wire (pts (xy 76.2 63.5) (xy 85.09 63.5))
+    (stroke (width 0) (type default) (color 0 0 0 0))
+  )
+  (wire (pts (xy 121.92 100.33) (xy 113.03 100.33))
+    (stroke (width 0) (type default) (color 0 0 0 0))
+  )
+  (wire (pts (xy 127 104.14) (xy 113.03 104.14))
+    (stroke (width 0) (type default) (color 0 0 0 0))
+  )
+  (wire (pts (xy 121.92 71.12) (xy 113.03 71.12))
+    (stroke (width 0) (type default) (color 0 0 0 0))
+  )
   (wire (pts (xy 121.92 66.04) (xy 113.03 66.04))
     (stroke (width 0) (type default) (color 0 0 0 0))
   )
-  (wire (pts (xy 121.92 73.66) (xy 113.03 73.66))
-    (stroke (width 0) (type default) (color 0 0 0 0))
-  )
-  (wire (pts (xy 121.92 81.28) (xy 113.03 81.28))
-    (stroke (width 0) (type default) (color 0 0 0 0))
-  )
-  (wire (pts (xy 121.92 60.96) (xy 113.03 60.96))
-    (stroke (width 0) (type default) (color 0 0 0 0))
-  )
-  (wire (pts (xy 83.82 166.37) (xy 91.44 166.37))
-    (stroke (width 0) (type default) (color 0 0 0 0))
-  )
-  (wire (pts (xy 76.2 86.36) (xy 85.09 86.36))
-    (stroke (width 0) (type default) (color 0 0 0 0))
-  )
-  (wire (pts (xy 218.44 60.96) (xy 209.55 60.96))
-    (stroke (width 0) (type default) (color 0 0 0 0))
-  )
-  (wire (pts (xy 121.92 97.79) (xy 113.03 97.79))
-    (stroke (width 0) (type default) (color 0 0 0 0))
-  )
-  (wire (pts (xy 74.93 104.14) (xy 85.09 104.14))
-    (stroke (width 0) (type default) (color 0 0 0 0))
-  )
-  (wire (pts (xy 74.93 101.6) (xy 85.09 101.6))
-    (stroke (width 0) (type default) (color 0 0 0 0))
-  )
-  (wire (pts (xy 74.93 66.04) (xy 85.09 66.04))
-    (stroke (width 0) (type default) (color 0 0 0 0))
-  )
-  (wire (pts (xy 218.44 55.88) (xy 209.55 55.88))
-    (stroke (width 0) (type default) (color 0 0 0 0))
-  )
-  (wire (pts (xy 77.47 74.93) (xy 85.09 74.93))
-    (stroke (width 0) (type default) (color 0 0 0 0))
-  )
-  (wire (pts (xy 121.92 88.9) (xy 113.03 88.9))
-    (stroke (width 0) (type default) (color 0 0 0 0))
-  )
-  (wire (pts (xy 83.82 171.45) (xy 91.44 171.45))
-    (stroke (width 0) (type default) (color 0 0 0 0))
-  )
-  (wire (pts (xy 180.34 78.74) (xy 189.23 78.74))
-    (stroke (width 0) (type default) (color 0 0 0 0))
-  )
-  (wire (pts (xy 118.11 135.89) (xy 105.41 135.89))
-    (stroke (width 0) (type default) (color 0 0 0 0))
-  )
-  (wire (pts (xy 180.34 53.34) (xy 189.23 53.34))
-    (stroke (width 0) (type default) (color 0 0 0 0))
-  )
-  (wire (pts (xy 180.34 68.58) (xy 189.23 68.58))
-    (stroke (width 0) (type default) (color 0 0 0 0))
-  )
-  (wire (pts (xy 76.2 63.5) (xy 85.09 63.5))
-    (stroke (width 0) (type default) (color 0 0 0 0))
-  )
-  (wire (pts (xy 121.92 100.33) (xy 113.03 100.33))
-    (stroke (width 0) (type default) (color 0 0 0 0))
-  )
-  (wire (pts (xy 127 104.14) (xy 113.03 104.14))
-    (stroke (width 0) (type default) (color 0 0 0 0))
-  )
-  (wire (pts (xy 121.92 71.12) (xy 113.03 71.12))
-    (stroke (width 0) (type default) (color 0 0 0 0))
-  )
-  (wire (pts (xy 121.92 55.88) (xy 113.03 55.88))
-    (stroke (width 0) (type default) (color 0 0 0 0))
-  )
   (wire (pts (xy 111.76 166.37) (xy 104.14 166.37))
     (stroke (width 0) (type default) (color 0 0 0 0))
@@
     (stroke (width 0) (type default) (color 0 0 0 0))
   )
+  (wire (pts (xy 121.92 63.5) (xy 113.03 63.5))
+    (stroke (width 0) (type default) (color 0 0 0 0))
+  )
+  (wire (pts (xy 121.92 95.25) (xy 113.03 95.25))
+    (stroke (width 0) (type default) (color 0 0 0 0))
+  )
+  (wire (pts (xy 189.23 99.06) (xy 196.85 99.06))
+    (stroke (width 0) (type default) (color 0 0 0 0))
+  )
+  (wire (pts (xy 104.14 171.45) (xy 111.76 171.45))
+    (stroke (width 0) (type default) (color 0 0 0 0))
+  )
+  (wire (pts (xy 76.2 81.28) (xy 85.09 81.28))
+    (stroke (width 0) (type default) (color 0 0 0 0))
+  )
+  (wire (pts (xy 180.34 55.88) (xy 189.23 55.88))
+    (stroke (width 0) (type default) (color 0 0 0 0))
+  )
+  (wire (pts (xy 85.09 99.06) (xy 74.93 99.06))
+    (stroke (width 0) (type default) (color 0 0 0 0))
+  )
+  (wire (pts (xy 208.28 120.65) (xy 213.36 120.65))
+    (stroke (width 0) (type default) (color 0 0 0 0))
+  )
   (wire (pts (xy 121.92 58.42) (xy 113.03 58.42))
     (stroke (width 0) (type default) (color 0 0 0 0))
   )
-  (wire (pts (xy 121.92 95.25) (xy 113.03 95.25))
-    (stroke (width 0) (type default) (color 0 0 0 0))
-  )
-  (wire (pts (xy 189.23 99.06) (xy 196.85 99.06))
-    (stroke (width 0) (type default) (color 0 0 0 0))
-  )
-  (wire (pts (xy 104.14 171.45) (xy 111.76 171.45))
-    (stroke (width 0) (type default) (color 0 0 0 0))
-  )
-  (wire (pts (xy 76.2 81.28) (xy 85.09 81.28))
-    (stroke (width 0) (type default) (color 0 0 0 0))
-  )
-  (wire (pts (xy 180.34 55.88) (xy 189.23 55.88))
-    (stroke (width 0) (type default) (color 0 0 0 0))
-  )
-  (wire (pts (xy 85.09 99.06) (xy 74.93 99.06))
-    (stroke (width 0) (type default) (color 0 0 0 0))
-  )
-  (wire (pts (xy 208.28 120.65) (xy 213.36 120.65))
-    (stroke (width 0) (type default) (color 0 0 0 0))
-  )
-  (wire (pts (xy 121.92 63.5) (xy 113.03 63.5))
-    (stroke (width 0) (type default) (color 0 0 0 0))
-  )
   (wire (pts (xy 180.34 76.2) (xy 189.23 76.2))
     (stroke (width 0) (type default) (color 0 0 0 0))
@@
     (effects (font (size 1.27 1.27)) (justify right bottom))
   )
-  (label "ROW_4" (at 121.92 58.42 180)
+  (label "ROW_4" (at 121.92 63.5 180)
     (effects (font (size 1.27 1.27)) (justify right bottom))
   )
@@
     (effects (font (size 1.27 1.27)) (justify right bottom))
   )
-  (label "ROW_5" (at 121.92 55.88 180)
-    (effects (font (size 1.27 1.27)) (justify right bottom))
-  )
-  (label "ROW_1" (at 121.92 66.04 180)
-    (effects (font (size 1.27 1.27)) (justify right bottom))
-  )
-  (label "ROW_2" (at 121.92 63.5 180)
+  (label "ROW_5" (at 121.92 66.04 180)
+    (effects (font (size 1.27 1.27)) (justify right bottom))
+  )
+  (label "ROW_1" (at 121.92 55.88 180)
+    (effects (font (size 1.27 1.27)) (justify right bottom))
+  )
+  (label "ROW_2" (at 121.92 58.42 180)
     (effects (font (size 1.27 1.27)) (justify right bottom))
   )
@@
       (reference "LED3") (unit 1) (value "SK6812MINI") (footprint "yuiop:SK6812MINI-E_B")
     )
-    (path "/00000000-0000-0000-0000-000060708fd9/00000000-0000-0000-0000-000060714969"
-      (reference "LED4") (unit 1) (value "SK6812MINI") (footprint "yuiop:SK6812MINI-E_B")
-    )
-    (path "/00000000-0000-0000-0000-000060708fd9/00000000-0000-0000-0000-0000607167db"
-      (reference "LED5") (unit 1) (value "SK6812MINI") (footprint "yuiop:SK6812MINI-E_B")
-    )
     (path "/00000000-0000-0000-0000-00006070a40a/00000000-0000-0000-0000-00006042e16a"
