File: yuiop32dm/main/yuiop32dm-main.kicad_pcb (KiCad board)
At the start: 2 copper layers, 166 x 116 mm, 114 parts, among them U1 ProMicro

Commit message: yuiop32dm: rev.1 finish
Parts:
- added C1: C, Capacitor_SMD:C_0603_1608Metric_Pad1.08x0.95mm_HandSolder, B.Cu at (144.5, 136.5)
- added C2: C, Capacitor_SMD:C_0603_1608Metric_Pad1.08x0.95mm_HandSolder, B.Cu at (144.5, 98.0)
- added H1: MountingHole_Pad, yuiop:Hole_2.2_4, F.Cu at (75.0, 51.0)
- added H2: MountingHole_Pad, yuiop:Hole_2.2_4, F.Cu at (225.0, 51.0)
- added H3: MountingHole_Pad, yuiop:Hole_2.2_4, F.Cu at (86.5, 141.5)
- added H4: MountingHole_Pad, yuiop:Hole_2.2_4, F.Cu at (213.5, 141.5)
- added H5: MountingHole_Pad, yuiop:Hole_2.2_4, F.Cu at (150.0, 100.0)
Connections:
- LED25 pad 2: unconnected-(LED25-Pad2) -> GND
- LED26 pad 2: unconnected-(LED26-Pad2) -> GND
- LED27 pad 2: unconnected-(LED27-Pad2) -> GND
- LED28 pad 2: unconnected-(LED28-Pad2) -> GND
- LED29 pad 2: unconnected-(LED29-Pad2) -> GND
- LED30 pad 2: unconnected-(LED30-Pad2) -> GND
- LED31 pad 2: unconnected-(LED31-Pad2) -> GND
Routing:
- net /LED: track 123.0 -> 119.2 mm
- net Net-(D9-Pad2): track 65.6 -> 63.5 mm
- net Net-(D13-Pad2): track 108.3 -> 106.3 mm
- net VCC: track 734.9 -> 733.0 mm
- net Net-(D5-Pad2): track 53.5 -> 51.6 mm
- net Net-(D1-Pad2): track 40.4 -> 38.5 mm
- net Net-(D12-Pad2): track 73.3 -> 72.6 mm
- net Net-(D8-Pad2): track 58.0 -> 57.4 mm
- net Net-(D29-Pad1): track 99.7 -> 99.1 mm
- net Net-(D30-Pad1): track 85.5 -> 84.8 mm
- net Net-(D4-Pad2): track 42.8 -> 42.2 mm
- net Net-(D31-Pad1): track 70.9 -> 70.3 mm
- net Net-(D26-Pad1): track 68.0 -> 67.5 mm
Other:
- board text added: "JLCJLCJLCJLC"
- board text added: "YUIOP32DM"
- board text added: "designed by KoRoN/KaoriYa"
- board text added: "revision 1"
