File: yuiop32dm/main/yuiop32dm-main.kicad_sch (KiCad schematic)
At the start: 114 parts, among them U1 ProMicro

Commit message: yuiop32dm: rev.1 finish
Parts:
- added C1, C2: C, Capacitor_SMD:C_0603_1608Metric_Pad1.08x0.95mm_HandSolder, symbol Device:C
- added H1, H2, H3, H4, H5: MountingHole_Pad, yuiop:Hole_2.2_4, symbol Mechanical:MountingHole_Pad
Connections:
- net GND: now also LED25.2 (GND), LED26.2 (GND), LED27.2 (GND), LED28.2 (GND), LED29.2 (GND), LED30.2 (GND), LED31.2 (GND), C1.2, C2.2, H1.1, H2.1, H3.1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
- net VCC: now also C1.1, C2.1
