File: yuiopPD/yuiopPD.kicad_sch (KiCad schematic)
At the start: 11 parts, among them J1 Keyball, J2 UART, J3 DEBUG, SW1 SW_Push, SW2 SW_Push, SW3 SW_Push, SW4 SW_Push, SW5 SW_Push, SW6 SW_Push, U1 SeeeduinoXIAO

Commit message: yuiopPD: finish grand design
Parts:
- added H1, H2, H3, H4, H5, H6, H7, H8, H9: MountingHole, MountingHole:MountingHole_2.1mm, symbol Mechanical:MountingHole
- added J4: OLED, yuiop:OLED_128x32, symbol Connector_Generic:Conn_01x04
- J1: footprint Connector_PinHeader_2.54mm:PinHeader_1x07_P2.54mm_Vertical -> yuiop:KeyballSensor_on_PCB
Connections:
- net +3V3: now also J4.3 (Pin_3)
- net GND: now also J2.1 (Pin_1), J4.4 (Pin_4); no longer J2.4 (Pin_4)
- net UART_TX: now also J2.4 (Pin_4); no longer J2.1 (Pin_1)
- net SCL: now reaches SW6.2, U1.6 (PA9_A5_D5_SCL)
- net SCL: now also J4.2 (Pin_2)
- net SDA: now reaches SW5.2, U1.5 (PA8_A4_D4_SDA)
- net SDA: now also J4.1 (Pin_1)
Other:
- moved on the sheet: J1, J2, J3, RST1, SW1, SW2, SW3, SW4, SW5, SW6, U1
