File: yuiopPD/main2/yuiopPD_r2.kicad_pcb (KiCad board)
At the start: 2 copper layers, 160 x 40 mm, 18 parts, among them J1 Keyball, J2 UART, J4 OLED, SW1 SW_Push, SW2 SW_Push, SW3 SW_Push, SW4 SW_Push, SW5 SW_Push, U1 Seeed Studio XIAO

Commit message: yuiopPD-r2: refine, finish, and generate production files
Parts:
- added H10: MountingHole, MountingHole:MountingHole_2.1mm, F.Cu at (93.0, 83.0)
- added H11: MountingHole, MountingHole:MountingHole_2.1mm, F.Cu at (93.0, 117.0)
- added H12: MountingHole, MountingHole:MountingHole_2.1mm, F.Cu at (183.0, 83.0)
- added H13: MountingHole, MountingHole:MountingHole_2.1mm, F.Cu at (183.0, 117.0)
- J2: footprint Connector_PinHeader_2.54mm:PinHeader_1x04_P2.54mm_Vertical -> Connector_PinHeader_2.54mm:PinHeader_1x02_P2.54mm_Vertical
- U1: value Seeed Studio XIAO -> SeeeduinoXIAO
- moved H2 13.5 mm to (109.5, 83.0)
- moved H7 13.5 mm to (109.5, 117.0)
- moved H3 11.0 mm to (145.5, 83.0)
- moved H8 11.0 mm to (145.5, 117.0)
- moved J2 5.00 mm to (84.0, 117.3)
- moved SW1 2.50 mm to (105.0, 100.0)
- moved J4 0.50 mm to (83.0, 82.3)
Connections:
- J2 pad 2: unconnected-(J2-Pad2) -> /UART_TX
Routing:
- net +3V3: track 165.0 -> 181.6 mm, vias 2 -> 0
- net /MOSI: track 160.0 -> 164.6 mm
- net /SDA: track 32.1 -> 35.0 mm
- net Net-(SW1-Pad2): track 45.7 -> 48.2 mm
- net /SCL: track 29.9 -> 31.4 mm
- net GND: vias 3 -> 0
