File: yuiopPD/main2/yuiopPD_r2.kicad_sch (KiCad schematic)
At the start: 18 parts, among them J1 Keyball, J2 UART, J4 OLED, SW1 SW_Push, SW2 SW_Push, SW3 SW_Push, SW4 SW_Push, SW5 SW_Push, U1 SeeeduinoXIAO

Commit message: yuiopPD-r2: refine, finish, and generate production files
Parts:
- added H10, H11, H12, H13: MountingHole, MountingHole:MountingHole_2.1mm, symbol Mechanical:MountingHole
- J2: footprint Connector_PinHeader_2.54mm:PinHeader_1x04_P2.54mm_Vertical -> Connector_PinHeader_2.54mm:PinHeader_1x02_P2.54mm_Vertical; symbol Connector_Generic:Conn_01x04 -> Connector_Generic:Conn_01x02
Connections:
- net UART_TX: now also J2.2 (Pin_2); no longer J2.4 (Pin_4)
- no-connect marks 7 -> 5
Other:
- moved on the sheet: H1, H2, H3, H4, H5, H6, H7, H8, H9
