File: yuiop60hh/topplate5-metal2-gasket/topplate5-metal2-gasket.kicad_pcb (KiCad board)
At the start: 2 copper layers, 294 x 104 mm, 60 parts

Commit message: fix
Other:
- board size 294 x 104 mm -> 295 x 104 mm
