File: yuiop2040C/yuiop2040C.kicad_pcb (KiCad board)
At the start: 2 copper layers, 15.7 x 31.5 mm, 31 parts, among them J1 Conn_01x20, J2 Conn_01x20, J3 Conn_01x03, U1 RP2040, U2 W25Q16JVSS, U3 MIC5219-3.3YM5, Y1 FA238V 12.000000MHz 10.0 +50.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

Commit message: fix
Parts:
- C1, C12, C13, C14, C2, C3, C4, C5, C6, C7, C8, C9: footprint Capacitor_SMD:C_0603_1608Metric -> Capacitor_SMD:C_0402_1005Metric
- R1, R2, R3, R4, R5, R6: footprint Resistor_SMD:R_0603_1608Metric -> Resistor_SMD:R_0402_1005Metric
- moved C15 58.4 mm to (78.0, 53.2), turned to 90 degrees
- moved C12 57.6 mm to (80.8, 76.9), turned to 90 degrees
- moved C16 56.4 mm to (83.1, 53.2), turned to 90 degrees
- moved R6 53.0 mm to (79.5, 57.4), turned to 90 degrees
- moved C13 52.9 mm to (85.4, 78.1), turned to 90 degrees
- moved R1 52.7 mm to (86.4, 61.1), turned to 90 degrees
- moved R5 50.2 mm to (79.5, 60.4), turned to 90 degrees
- moved C14 48.0 mm to (86.4, 57.3), turned to -90 degrees
- moved R3 43.2 mm to (85.4, 76.1), turned to 90 degrees
- moved R4 42.9 mm to (88.9, 79.4), turned to 90 degrees
- moved R2 40.1 mm to (87.9, 61.1), turned to 90 degrees
- moved C11 29.0 mm to (121.5, 67.4)
- moved C10 24.9 mm to (117.7, 67.4)
- moved C17 17.6 mm to (114.1, 77.0)
- moved U2 16.1 mm to (82.9, 58.9), turned to 90 degrees
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Routing:
- net GND: track 0.00 -> 59.6 mm, vias 0 -> 1
- net +3V3: track 0.00 -> 43.5 mm, vias 0 -> 3
- net /VSYS: track 0.00 -> 16.3 mm
- net /SWCLK: track 0.00 -> 15.6 mm, vias 0 -> 2
- net /SWD: track 0.00 -> 12.0 mm
- net /GPIO15: track 0.00 -> 11.7 mm
- net /GPIO14: track 0.00 -> 10.3 mm
- net /QSPI_SD3: track 0.00 -> 9.69 mm, vias 0 -> 2
- net /QSPI_SD0: track 0.00 -> 9.60 mm
- net /QSPI_SCLK: track 0.00 -> 9.09 mm, vias 0 -> 2
- net /GPIO16: track 0.00 -> 8.91 mm
- net /GPIO13: track 0.00 -> 8.84 mm
- net /RUN: track 0.00 -> 8.55 mm
- net /GPIO17: track 0.00 -> 7.47 mm
- net /GPIO12: track 0.00 -> 7.41 mm
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Other:
- board size 15.7 x 31.5 mm -> 15.7 x 34.6 mm
