File: rp2040-controller/rp2040-controller.kicad_sch (KiCad schematic)
At the start: 34 parts, among them J1 USB_C_Receptacle_USB2.0, J5 Conn_01x03, U1 RP2040, U2 W25Q16JVSS, U3 MIC5219-3.3YM5, Y1 FA238V 12.000000MHz 10.0 +50.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

Commit message: convert for KiCad 8
Parts:
- F1: value MF-NSMF050-2 -> Fuse_Small; footprint Fuse:Fuse_1206_3216Metric -> (none)
- J1: value USB_C_Receptacle_USB2.0 -> USB_C_Receptacle_USB2.0_16P; footprint Connector_USB:USB_C_Receptacle_XKB_U262-16XN-4BVC11 -> (none); symbol Connector:USB_C_Receptacle_USB2.0 -> Connector:USB_C_Receptacle_USB2.0_16P
- U1: footprint RP2040_minimal:RP2040-QFN-56-r2 -> RP2040_minimal:RP2040-QFN-56
- U2: value W25Q16JVSS -> W25Q32JVSS; footprint Package_SO:SOIC-8_3.9x4.9mm_P1.27mm -> Package_SO:SOIC-8_5.23x5.23mm_P1.27mm
Other:
- moved on the sheet: C17, C4, C5, R3, R4, R6, U2, Y1
