File: yuiop29re/yuiop29re-topplate.kicad_pcb (KiCad board)
At the start: 2 copper layers, 118 x 118 mm, 29 parts

Commit message: yuiop29re: add JLC serial position mark
Other:
- board text added: "JLCJLCJLCJLC"
Changed lines of the file:
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@@
 		(layer "Edge.Cuts")
+	)
+	(gr_text "JLCJLCJLCJLC"
+		(at 101.2 157.4 0)
+		(layer "B.SilkS")
+		(effects
+			(font
+				(size 0.8 0.8)
+				(thickness 0.15)
+			)
+			(justify left bottom mirror)
+		)
 	)
 	(gr_text "RESET"
@@
 		(polygon
 			(pts
-				(xy 208.5 41.5) (xy 209 159) (xy 91.5 158.5) (xy 91 41)
+				(xy 209 41) (xy 209 159) (xy 91 159) (xy 91 41)
 			)
 		)
@@
 		(polygon
 			(pts
-				(xy 91 41) (xy 208.5 41.5) (xy 209 159) (xy 91.5 158.5)
-			)
-		)
+				(xy 91 41) (xy 209 41) (xy 209 159) (xy 91 159)
+			)
+		)

Commit message: yiuop29re: add product marks
Other:
- board text added: "YUIOP29RE"
- board text added: "designed by KoRoN/KaoriYa"
- board text added: "revision 1"
