File: yuiop29re/yuiop29re-topplate.kicad_pcb (KiCad board)
At the start: 2 copper layers, 118 x 118 mm, 29 parts

Commit message: revise yuiop29re
Parts:
- added HOLE**: Hole_3.6, yuiop:Hole_3.6, F.Cu at (96.0, 46.5)
- added HOLE**: Hole_2.2, yuiop:Hole_2.2, F.Cu at (196.4, 55.5)
- added HOLE**: Hole_3.6, yuiop:Hole_3.6, F.Cu at (203.5, 153.5)
- added HOLE**: Hole_2.2, yuiop:Hole_2.2, F.Cu at (202.5, 56.0)
- added HOLE**: Hole_3.6, yuiop:Hole_3.6, F.Cu at (203.5, 46.5)
- added HOLE**: Hole_2.2, yuiop:Hole_2.2, F.Cu at (97.5, 56.0)
- added HOLE**: Hole_2.2, yuiop:Hole_2.2, F.Cu at (97.5, 144.0)
- added HOLE**: Hole_2.2, yuiop:Hole_2.2, F.Cu at (202.5, 144.0)
- added HOLE**: Hole_3.6, yuiop:Hole_3.6, F.Cu at (96.5, 153.5)
- added HOLE**: Hole_2.2, yuiop:Hole_2.2, F.Cu at (150.0, 100.0)
- added HOLE**: Hole_2.2, yuiop:Hole_2.2, F.Cu at (196.4, 49.5)
- KSW1, KSW10, KSW11, KSW12, KSW13, KSW14, KSW15, KSW16, KSW17, KSW18, KSW19, KSW2, KSW20, KSW21, KSW22, KSW23, KSW24, KSW25, KSW26, KSW27, KSW28, KSW29, KSW3, KSW4, KSW5, KSW6, KSW7, KSW8, KSW9: footprint yuiop:TopPlate_v2_Switch_1u -> yuiop:TopPlate_v3_Switch_1u
Other:
- outline, holes or cut-outs redrawn
- board text added: "revision 2"
- board text removed: "revision 1"
