File: yuiop29re/yuiop29re.kicad_pcb (KiCad board)
At the start: 2 copper layers, 116.5 x 116.5 mm, 123 parts, among them J1 USB_C_Receptacle_USB2.0_16P, J2 SSD1306 OLED, J3 MJ-4PP-9, J4 UART0, J5 SWD, Q1 BSS138, U1 RP2040_breakout

Commit message: revise yuiop29re
Parts:
- moved C6 1.27 mm to (159.2, 51.1)
- moved R10 1.27 mm to (159.2, 48.1)
- moved R9 1.27 mm to (159.2, 45.0)
- moved J5 0.41 mm to (128.0, 45.1)
- moved J4 0.30 mm to (137.0, 45.1)
- moved J3 0.24 mm to (165.0, 47.8)
Routing:
- net GND: track 881.4 -> 883.0 mm
- net /3V3: track 133.1 -> 134.2 mm
- net /I2C1_SCLK: track 34.2 -> 35.0 mm
- net /I2C1_SDA: track 34.5 -> 35.3 mm
- net /5V0: track 780.4 -> 779.9 mm
Other:
- board text added: "revision 1.1"
- board text removed: "revision 1"
